File: XO-Stick2.sch (EAGLE design)
At the start: 31 parts, among them J1 POWER, J2 85MOTR, J3 85MOTL, J4 REF, J5 SCL, J6 SDA, J7 AVCC (N/C), J8 AGND (N/C), J9 EXT VCC, SW1 USER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

Commit message: XO Stick v14: move USB to PB3/4 (Louis Beaudoin suggestion).
This allows more straightforward use of the XO Stick as a programmer,
and of the XO Stick's I2C bus.

It complicates use of the '85 to drive the XOrduino bot, but that's probably
a reasonable sacrifice.
Parts:
- removed J2: 85MOTR, xorduino:JUMPER-2SJ-NO
- removed J3: 85MOTL, xorduino:JUMPER-2SJ-NO
- removed J5: SCL, xorduino:JUMPER-2SJ-NC-BOT
- removed J6: SDA, xorduino:JUMPER-2SJ-NC-BOT
- J1: device xorduino:JUMPER-3WAYTRACE-NOCONFLICT -> xorduino:JUMPER-4WAY
Connections:
- removed net D_M: H2.4, J6.2, R2.2, U1.(MOSI)PB0, U2.(MOSI/DI/SDA/!OC1A!)PB0
- removed net D_P: H2.3, J5.2, R1.2, U1.(SCK)PB2, U2.(SCK/SCL/!OC1B!)PB2
- removed net SCL: H1.SCL, J5.1
- removed net SDA: H1.SDA, J6.1
- new net ARD_3.3V: H1.3.3V, J1.N/O2
- new net PB0: H1.D13, H1.D2, H1.SDA, H2.4, R4.2, U1.(MOSI)PB0, U2.(MOSI/DI/SDA/!OC1A!)PB0
- new net PB2: H1.*D3, H1.D12, H1.SCL, H2.3, SW1.1, U1.(SCK)PB2, U2.(SCK/SCL/!OC1B!)PB2
- net ARD_5V: now also J1.N/O1; no longer J1.N/O
- net PA2: now also JP1.4
- net PA5: no longer J2.1
- net PB1: now also R5.2; no longer R4.2
- net PB3: now also R2.2; no longer H1.*D10, R5.2
- net PB4: now also R1.2; no longer H1.D12, J2.2, J3.1, JP1.4, SW1.1
- net PB5: now also H1.*D10; no longer H1.*D9
- net PB6: no longer J3.2
Other:
- note added: "14"
- note removed: "(needs to be closed to program XO Stick from XOrduino)"
- note removed: "13"
- note removed: "Close jumpers to drive motors from '85"
- note removed: "Open N/C jumpers to separate I2C from USB"
- moved on the sheet: J4, U1
