File: XO-Tester.brd (EAGLE design)
At the start: 55.9 x 53.3 mm, 39 parts, among them SW1 RESET

Commit message: Gerbers for the test shield.
Parts:
- moved JP1 30.7 mm to (49.5, 24.8)
- moved JP2 24.2 mm to (49.5, 27.3)
- moved JP3 17.8 mm to (49.5, 29.8)
- moved RN1 4.49 mm to (36.2, 25.4)
- moved RN2 4.45 mm to (14.6, 25.4)
- moved RN4 3.24 mm to (36.2, 29.2)
- moved RN3 3.17 mm to (14.6, 29.2)
- moved LED10 2.54 mm to (19.1, 18.4)
- moved LED11 2.54 mm to (25.4, 18.4)
- moved LED12 2.54 mm to (31.8, 18.4)
- moved LED13 2.54 mm to (38.1, 18.4)
- moved LED14 2.54 mm to (44.5, 18.4)
- moved LED8 2.54 mm to (6.35, 18.4)
- moved LED9 2.54 mm to (12.7, 18.4)
- moved LED22 1.27 mm to (6.35, 35.6)
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Routing:
- net USER2: track 10.8 -> 80.6 mm, vias 0 -> 4
- net N$19: track 29.9 -> 94.2 mm, vias 2 -> 7
- net N$24: track 27.9 -> 91.7 mm, vias 0 -> 3
- net N$20: track 24.6 -> 67.0 mm, vias 1 -> 3
- net USER1: track 11.2 -> 49.3 mm, vias 0 -> 3
- net A0: track 59.2 -> 23.2 mm, vias 2 -> 1
- net D5: track 51.7 -> 23.5 mm
- net N$9: track 25.5 -> 46.0 mm, vias 1 -> 4
- net N$21: track 38.0 -> 58.3 mm, vias 2 -> 6
- net N$8: track 24.0 -> 39.7 mm
- net N$10: track 17.2 -> 31.7 mm, vias 0 -> 1
- net D7: track 25.3 -> 38.4 mm, vias 1 -> 0
- net USER3: track 11.9 -> 20.7 mm
- net N$18: track 26.3 -> 19.2 mm
- net N$23: track 32.0 -> 25.7 mm, vias 1 -> 0
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Other:
- board text added: "1"
- board text added: "2"
- board text added: "3"
- board text added: "IOREF"
- board text added: "USER"
- board text added: "USER1"
- board text added: "USER2"
- board text added: "USER3"
